File: switch_button_tester.kicad_sch (KiCad schematic)
At the start: 0 parts

Commit message: progress
Parts:
- added D1: LED, LED_SMD:LED_0603_1608Metric_Pad1.05x0.95mm_HandSolder, symbol Device:LED
- added J1: Conn_01x02_Pin, Connector_PinHeader_2.54mm:PinHeader_1x02_P2.54mm_Vertical_SMD_Pin1Left, symbol Connector:Conn_01x02_Pin
- added R1: 100, Resistor_SMD:R_0603_1608Metric_Pad0.98x0.95mm_HandSolder, symbol Device:R
- added SW1, SW2: SW_Push, MX_Hotswap:MX-Hotswap-1U, symbol Switch:SW_Push
- added SW3, SW4: SW_Push, Button_Switch_Keyboard:SW_Cherry_MX_1.00u_PCB, symbol Switch:SW_Push
Connections:
- new net: J1.2 (Pin_2), SW1.1, SW2.1, SW3.1, SW4.1
- new net: D1.2 (A), SW1.2, SW2.2, SW3.2, SW4.2
- new net: J1.1 (Pin_1), R1.1
- new net: D1.1 (K), R1.2
